File: EGR226 Project.sch (EAGLE design)
At the start: 0 parts

Commit message: schematic complete, fix interupt components are complete
Parts:
- added 2N700, 2N7000: IRF510, transistor-fet:IRF510
- added GREEN, RED: (no value), eagle-ltspice:LED_ELD260
- added KEYPAD1: KEYPAD, Keypad:KEYPAD
- added LCD1: LCD, LCD:LCD
- added MOTOR1: DC_MOTOR, Motor:DC_MOTOR
- added OK1: IL5, optocoupler:IL5
- added R1: 470, resistor:R-US_0204/5
- added R10: 100, resistor:R-US_0204/5
- added R3: 220, resistor:R-US_0204/5
- added RGB_LED: GM1WA55311A, led:GM1WA55311A
- added SERVO1: (no value), Servo:SERVO
- added SWITCH-TACTILE: (no value), switch-omron:10-XX
Connections:
- new net +3V3: MOTOR1.V_IN
- new net +5V: LCD1.VDD, R1.2, R10.2, R3.2, SERVO1.+5V
- new net GND: 2N700.S, 2N7000.S, LCD1.RW, LCD1.VSS, OK1.C, OK1.EMI, RGB_LED.A, SERVO1.GND, SWITCH-TACTILE.S
- new net N$1: SERVO1.SIGNAL
- new net N$10: LCD1.VO
- new net N$11: KEYPAD1.1
- new net N$12: KEYPAD1.2
- new net N$13: KEYPAD1.3
- new net N$14: KEYPAD1.4
- new net N$15: KEYPAD1.5
- new net N$16: KEYPAD1.6
- new net N$17: KEYPAD1.7
- new net N$18: RGB_LED.CRED
- new net N$19: RGB_LED.CBLUE
- new net N$2: OK1.A
- new net N$20: RGB_LED.CGREEN
- new net N$21: 2N700.G
- new net N$22: 2N7000.G
- new net N$23: SWITCH-TACTILE.P
- new net N$24: R1.1, R3.1, RED.A
- new net N$25: 2N7000.D, RED.C
- new net N$27: 2N700.D, GREEN.C
- new net N$28: GREEN.A, R10.1
- new net N$3: MOTOR1.GND, OK1.COL
- new net N$4: LCD1.E
- new net N$5: LCD1.RS
- new net N$6: LCD1.DB4
- new net N$7: LCD1.DB5
- new net N$8: LCD1.DB6
- new net N$9: LCD1.DB7
Other:
- note added: "2N7000"
- note removed: "Fan with E-stop"
- note removed: "KeyPad"
- note removed: "LCD"
- note removed: "RGB and turnoff"
- note removed: "RW/E"
- note removed: "Servo w/ Red/Green LED"
- note removed: "Timer_A"
- note removed: "contrast"
- note removed: "data"

Commit message: Fully Fuctional Minimum Reqirments!
Parts:
- added R2, R4: 100, resistor:R-US_0204/5
- added R5: 160, resistor:R-US_0204/7
Connections:
- new net N$26: R5.2
- new net N$29: R5.1, RGB_LED.CBLUE
- new net N$30: R4.1, RGB_LED.CGREEN
- net N$18: now also R2.2; no longer RGB_LED.CRED
- net N$19: now also R2.1, RGB_LED.CRED; no longer RGB_LED.CBLUE
- net N$20: now also R4.2; no longer RGB_LED.CGREEN
Other:
- note added: "Blue"
- note added: "Green"
- note added: "Red"
- moved on the sheet: RGB_LED
Changed lines of the file:
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@@
 <part name="SWITCH-TACTILE" library="switch-omron" library_urn="urn:adsk.eagle:library:377" deviceset="10-XX" device=""/>
 <part name="SUPPLY8" library="supply2" library_urn="urn:adsk.eagle:library:372" deviceset="GND" device=""/>
+<part name="R2" library="resistor" library_urn="urn:adsk.eagle:library:348" deviceset="R-US_" device="0204/5" value="100"/>
+<part name="R4" library="resistor" library_urn="urn:adsk.eagle:library:348" deviceset="R-US_" device="0204/5" value="100"/>
+<part name="R5" library="resistor" library_urn="urn:adsk.eagle:library:348" deviceset="R-US_" device="0204/7" value="160"/>
 </parts>
 <sheets>
@@
 <text x="54.356" y="-64.516" size="1.778" layer="91">2N7000</text>
 <text x="33.782" y="-64.262" size="1.778" layer="91">2N7000</text>
+<text x="-22.86" y="43.18" size="1.778" layer="91" rot="R90">Blue</text>
+<text x="-17.78" y="43.18" size="1.778" layer="91" rot="R90">Red</text>
+<text x="-12.7" y="40.64" size="1.778" layer="91" rot="R90">Green</text>
 </plain>
 <moduleinsts>
@@
 <attribute name="VALUE" x="-64.135" y="8.255" size="1.778" layer="96" rot="R180"/>
 </instance>
-<instance part="RGB_LED" gate="G$1" x="-17.78" y="50.8" smashed="yes">
-<attribute name="NAME" x="-20.32" y="51.562" size="1.778" layer="95"/>
+<instance part="RGB_LED" gate="G$1" x="-17.78" y="53.34" smashed="yes">
+<attribute name="NAME" x="-20.32" y="54.102" size="1.778" layer="95"/>
 </instance>
 <instance part="SUPPLY6" gate="GND" x="-22.86" y="60.96" rot="R180"/>
@@
 <instance part="SWITCH-TACTILE" gate="1" x="40.64" y="-7.62" rot="R270"/>
 <instance part="SUPPLY8" gate="GND" x="50.8" y="-7.62" rot="R90"/>
+<instance part="R2" gate="G$1" x="-22.86" y="35.56" smashed="yes" rot="R270">
+<attribute name="VALUE" x="-26.162" y="39.37" size="1.778" layer="96" rot="R270"/>
+</instance>
+<instance part="R4" gate="G$1" x="-12.7" y="35.56" smashed="yes" rot="R270">
+<attribute name="VALUE" x="-16.002" y="39.37" size="1.778" layer="96" rot="R270"/>
+</instance>
+<instance part="R5" gate="G$1" x="-17.78" y="35.56" smashed="yes" rot="R270">
+<attribute name="VALUE" x="-21.082" y="39.37" size="1.778" layer="96" rot="R270"/>
+</instance>
 </instances>
 <busses>
@@
 <pinref part="SUPPLY6" gate="GND" pin="GND"/>
 <pinref part="RGB_LED" gate="G$1" pin="A"/>
-<wire x1="-22.86" y1="58.42" x2="-22.86" y2="53.34" width="0.1524" layer="91"/>
+<wire x1="-22.86" y1="58.42" x2="-22.86" y2="55.88" width="0.1524" layer="91"/>
 </segment>
 <segment>
@@
 <net name="N$18" class="0">
 <segment>
-<pinref part="RGB_LED" gate="G$1" pin="CRED"/>
 <portref moduleinst="MSP432-1" port="P2.4"/>
 <wire x1="-20.32" y1="22.86" x2="-22.86" y2="22.86" width="0.1524" layer="91"/>
-<wire x1="-22.86" y1="22.86" x2="-22.86" y2="45.72" width="0.1524" layer="91"/>
-</segment>
-</net>
-<net name="N$19" class="0">
-<segment>
-<portref moduleinst="MSP432-1" port="P2.5"/>
-<pinref part="RGB_LED" gate="G$1" pin="CBLUE"/>
-<wire x1="-17.78" y1="22.86" x2="-17.78" y2="45.72" width="0.1524" layer="91"/>
+<pinref part="R2" gate="G$1" pin="2"/>
+<wire x1="-22.86" y1="22.86" x2="-22.86" y2="30.48" width="0.1524" layer="91"/>
 </segment>
 </net>
@@
 <portref moduleinst="MSP432-1" port="P2.6"/>
 <wire x1="-15.24" y1="22.86" x2="-12.7" y2="22.86" width="0.1524" layer="91"/>
-<pinref part="RGB_LED" gate="G$1" pin="CGREEN"/>
-<wire x1="-12.7" y1="22.86" x2="-12.7" y2="45.72" width="0.1524" layer="91"/>
+<pinref part="R4" gate="G$1" pin="2"/>
+<wire x1="-12.7" y1="22.86" x2="-12.7" y2="30.48" width="0.1524" layer="91"/>
 </segment>
 </net>
@@
 </segment>
 </net>
+<net name="N$19" class="0">
+<segment>
+<pinref part="R2" gate="G$1" pin="1"/>
+<pinref part="RGB_LED" gate="G$1" pin="CRED"/>
+<wire x1="-22.86" y1="40.64" x2="-22.86" y2="48.26" width="0.1524" layer="91"/>
+</segment>
+</net>
+<net name="N$26" class="0">
+<segment>
+<pinref part="R5" gate="G$1" pin="2"/>
+<portref moduleinst="MSP432-1" port="P2.5"/>
+<wire x1="-17.78" y1="22.86" x2="-17.78" y2="30.48" width="0.1524" layer="91"/>
+</segment>
+</net>
+<net name="N$29" class="0">
+<segment>
+<pinref part="R5" gate="G$1" pin="1"/>
+<pinref part="RGB_LED" gate="G$1" pin="CBLUE"/>
+<wire x1="-17.78" y1="40.64" x2="-17.78" y2="48.26" width="0.1524" layer="91"/>
+</segment>
+</net>
+<net name="N$30" class="0">
+<segment>
+<pinref part="R4" gate="G$1" pin="1"/>
+<pinref part="RGB_LED" gate="G$1" pin="CGREEN"/>
+<wire x1="-12.7" y1="40.64" x2="-12.7" y2="48.26" width="0.1524" layer="91"/>
+</segment>
+</net>

Commit message: Finished Schematic
Parts:
- added R6, R7: 100, resistor:R-US_0204/5
- added R8, R9: 56, resistor:R-US_0204/5
- added SP1, SP2: AL11P, buzzer:AL11P
- added SWITCH-TACTILE_2: (no value), switch-omron:10-XX
- added T1, T4: TIP31C, transistor-neu-to92:TIP31C
Connections:
- new net N$31: SWITCH-TACTILE_2.P
- new net N$32: R6.1, R8.2
- new net N$33: R7.1, R9.2
- new net N$34: T1.B
- new net N$35: T4.B
- new net N$36: R9.1, T4.C
- new net N$37: SP2.1, T4.E
- new net N$38: SP1.1, T1.E
- new net N$39: R8.1, T1.C
- net +3V3: now also R6.2, R7.2
- net GND: now also SP1.2, SP2.2, SWITCH-TACTILE_2.S

Commit message: Final Product 1e
Connections:
- net GND: now also T1.E, T4.E; no longer SP1.2, SP2.2
- net N$36: now also R8.1, SP1.1; no longer R9.1, T4.C
- net N$37: now also SP1.2, T1.C; no longer SP2.1, T4.E
- net N$38: now also R9.1, SP2.1; no longer SP1.1, T1.E
- net N$39: now also SP2.2, T4.C; no longer R8.1, T1.C
Other:
- moved on the sheet: SP1, SP2
Changed lines of the file:
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@@
 <attribute name="VALUE" x="57.15" y="56.642" size="1.778" layer="96" rot="R180"/>
 </instance>
-<instance part="SP1" gate="G$1" x="83.82" y="71.12" smashed="yes">
-<attribute name="NAME" x="80.01" y="77.47" size="1.778" layer="95"/>
+<instance part="SP1" gate="G$1" x="68.58" y="71.12" smashed="yes">
+<attribute name="NAME" x="64.77" y="77.47" size="1.778" layer="95"/>
 </instance>
-<instance part="SP2" gate="G$1" x="83.82" y="53.34" smashed="yes">
-<attribute name="NAME" x="80.01" y="59.69" size="1.778" layer="95"/>
+<instance part="SP2" gate="G$1" x="68.58" y="53.34" smashed="yes">
+<attribute name="NAME" x="64.77" y="59.69" size="1.778" layer="95"/>
 </instance>
 <instance part="+3V2" gate="G$1" x="25.4" y="71.12" rot="R90"/>
 <instance part="+3V3" gate="G$1" x="25.4" y="53.34" rot="R90"/>
-<instance part="T4" gate="G$1" x="68.58" y="50.8" smashed="yes" rot="R90">
-<attribute name="VALUE" x="68.58" y="53.34" size="1.778" layer="96" rot="R90"/>
+<instance part="T4" gate="G$1" x="83.82" y="50.8" smashed="yes" rot="R90">
+<attribute name="VALUE" x="83.82" y="53.34" size="1.778" layer="96" rot="R90"/>
 </instance>
-<instance part="SUPPLY10" gate="GND" x="93.98" y="71.12" rot="R90"/>
-<instance part="T1" gate="G$1" x="68.58" y="68.58" smashed="yes" rot="R90">
-<attribute name="VALUE" x="68.58" y="71.12" size="1.778" layer="96" rot="R90"/>
+<instance part="SUPPLY10" gate="GND" x="96.52" y="71.12" rot="R90"/>
+<instance part="T1" gate="G$1" x="83.82" y="68.58" smashed="yes" rot="R90">
+<attribute name="VALUE" x="83.82" y="71.12" size="1.778" layer="96" rot="R90"/>
 </instance>
-<instance part="SUPPLY11" gate="GND" x="93.98" y="53.34" rot="R90"/>
+<instance part="SUPPLY11" gate="GND" x="96.52" y="53.34" rot="R90"/>
 </instances>
 <busses>
@@
 </segment>
 <segment>
-<pinref part="SP2" gate="G$1" pin="2"/>
+<pinref part="T1" gate="G$1" pin="E"/>
+<pinref part="SUPPLY10" gate="GND" pin="GND"/>
+<wire x1="88.9" y1="71.12" x2="93.98" y2="71.12" width="0.1524" layer="91"/>
+</segment>
+<segment>
+<pinref part="T4" gate="G$1" pin="E"/>
 <pinref part="SUPPLY11" gate="GND" pin="GND"/>
-<wire x1="88.9" y1="53.34" x2="91.44" y2="53.34" width="0.1524" layer="91"/>
-</segment>
-<segment>
-<pinref part="SP1" gate="G$1" pin="2"/>
-<pinref part="SUPPLY10" gate="GND" pin="GND"/>
-<wire x1="88.9" y1="71.12" x2="91.44" y2="71.12" width="0.1524" layer="91"/>
+<wire x1="88.9" y1="53.34" x2="93.98" y2="53.34" width="0.1524" layer="91"/>
 </segment>
 </net>
@@
 <portref moduleinst="MSP432-1" port="P7.6"/>
 <wire x1="20.32" y1="22.86" x2="20.32" y2="63.5" width="0.1524" layer="91"/>
+<wire x1="20.32" y1="63.5" x2="83.82" y2="63.5" width="0.1524" layer="91"/>
 <pinref part="T1" gate="G$1" pin="B"/>
-<wire x1="20.32" y1="63.5" x2="68.58" y2="63.5" width="0.1524" layer="91"/>
-<wire x1="68.58" y1="63.5" x2="68.58" y2="66.04" width="0.1524" layer="91"/>
+<wire x1="83.82" y1="63.5" x2="83.82" y2="66.04" width="0.1524" layer="91"/>
 </segment>
 </net>
@@
 <portref moduleinst="MSP432-1" port="P7.7"/>
 <wire x1="22.86" y1="22.86" x2="22.86" y2="43.18" width="0.1524" layer="91"/>
+<wire x1="22.86" y1="43.18" x2="83.82" y2="43.18" width="0.1524" layer="91"/>
 <pinref part="T4" gate="G$1" pin="B"/>
-<wire x1="22.86" y1="43.18" x2="68.58" y2="43.18" width="0.1524" layer="91"/>
-<wire x1="68.58" y1="43.18" x2="68.58" y2="48.26" width="0.1524" layer="91"/>
+<wire x1="83.82" y1="43.18" x2="83.82" y2="48.26" width="0.1524" layer="91"/>
 </segment>
 </net>
 <net name="N$36" class="0">
 <segment>
+<pinref part="R8" gate="G$1" pin="1"/>
+<pinref part="SP1" gate="G$1" pin="1"/>
+<wire x1="58.42" y1="71.12" x2="63.5" y2="71.12" width="0.1524" layer="91"/>
+</segment>
+</net>
+<net name="N$37" class="0">
+<segment>
+<pinref part="SP1" gate="G$1" pin="2"/>
+<pinref part="T1" gate="G$1" pin="C"/>
+<wire x1="73.66" y1="71.12" x2="78.74" y2="71.12" width="0.1524" layer="91"/>
+</segment>
+</net>
+<net name="N$38" class="0">
+<segment>
 <pinref part="R9" gate="G$1" pin="1"/>
+<pinref part="SP2" gate="G$1" pin="1"/>
+<wire x1="58.42" y1="53.34" x2="63.5" y2="53.34" width="0.1524" layer="91"/>
+</segment>
+</net>
+<net name="N$39" class="0">
+<segment>
+<pinref part="SP2" gate="G$1" pin="2"/>
 <pinref part="T4" gate="G$1" pin="C"/>
-<wire x1="58.42" y1="53.34" x2="63.5" y2="53.34" width="0.1524" layer="91"/>
-</segment>
-</net>
-<net name="N$37" class="0">
-<segment>
-<pinref part="T4" gate="G$1" pin="E"/>
-<pinref part="SP2" gate="G$1" pin="1"/>
 <wire x1="73.66" y1="53.34" x2="78.74" y2="53.34" width="0.1524" layer="91"/>
 </segment>
 </net>
-<net name="N$38" class="0">
-<segment>
-<pinref part="T1" gate="G$1" pin="E"/>
-<pinref part="SP1" gate="G$1" pin="1"/>
-<wire x1="73.66" y1="71.12" x2="78.74" y2="71.12" width="0.1524" layer="91"/>
-</segment>
-</net>
-<net name="N$39" class="0">
-<segment>
-<pinref part="R8" gate="G$1" pin="1"/>
-<pinref part="T1" gate="G$1" pin="C"/>
-<wire x1="58.42" y1="71.12" x2="63.5" y2="71.12" width="0.1524" layer="91"/>
-</segment>
-</net>
